File: filter.kicad_sch (KiCad schematic)
At the start: 24 parts

Commit message: intial version of pcb
Parts:
- C11, C12, C13, C14, C15, C16, C17, C18, C19, C20: footprint (none) -> joka:C_0805_2012Metric; symbol Device:C -> joka:C
- F1, F2: footprint (none) -> joka:Fuse_0805_2012Metric; symbol Device:Fuse -> joka:Fuse
- L1, L2, L3, L4, L5, L6, L7, L8: footprint (none) -> joka:L_0805_2012Metric; symbol Device:L -> joka:L
- R2, R3, R4, R5: footprint (none) -> joka:R_0805_2012Metric; symbol Device:R -> joka:R
Changed lines of the file:
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@@
 	)
 	(symbol
-		(lib_id "Device:L")
+		(lib_id "joka:L")
 		(at 127 85.09 0)
 		(unit 1)
@@
 			)
 		)
-		(property "Footprint" ""
+		(property "Footprint" "joka:L_0805_2012Metric"
 			(at 127 85.09 0)
 			(effects
@@
 	)
 	(symbol
-		(lib_id "Device:L")
+		(lib_id "joka:L")
 		(at 101.6 118.11 0)
 		(unit 1)
@@
 			)
 		)
-		(property "Footprint" ""
+		(property "Footprint" "joka:L_0805_2012Metric"
 			(at 101.6 118.11 0)
 			(effects
@@
 	)
 	(symbol
-		(lib_id "Device:C")
+		(lib_id "joka:C")
 		(at 54.61 165.1 90)
 		(unit 1)
@@
 			)
 		)
-		(property "Footprint" ""
+		(property "Footprint" "joka:C_0805_2012Metric"
 			(at 58.42 164.1348 0)
 			(effects
@@
 	)
 	(symbol
-		(lib_id "Device:Fuse")
+		(lib_id "joka:Fuse")
 		(at 194.31 127 90)
 		(unit 1)
@@
 			)
 		)
-		(property "Footprint" ""
+		(property "Footprint" "joka:Fuse_0805_2012Metric"
 			(at 194.31 128.778 90)
 			(effects
@@
 	)
 	(symbol
-		(lib_id "Device:C")
+		(lib_id "joka:C")
 		(at 63.5 85.09 0)
 		(unit 1)
@@
 			)
 		)
-		(property "Footprint" ""
+		(property "Footprint" "joka:C_0805_2012Metric"
 			(at 64.4652 88.9 0)
 			(effects
@@
 	)
 	(symbol
-		(lib_id "Device:L")
+		(lib_id "joka:L")
 		(at 54.61 76.2 90)
 		(unit 1)
@@
 			)
 		)
-		(property "Footprint" ""
+		(property "Footprint" "joka:L_0805_2012Metric"
 			(at 54.61 76.2 0)
 			(effects
@@
 	)
 	(symbol
-		(lib_id "Device:R")
+		(lib_id "joka:R")
 		(at 63.5 156.21 0)
 		(unit 1)
@@
 			)
 		)
-		(property "Footprint" ""
+		(property "Footprint" "joka:R_0805_2012Metric"
 			(at 61.722 156.21 90)
 			(effects
@@
 	)
 	(symbol
-		(lib_id "Device:L")
+		(lib_id "joka:L")
 		(at 156.21 127 90)
 		(unit 1)
@@
 			)
 		)
-		(property "Footprint" ""
+		(property "Footprint" "joka:L_0805_2012Metric"
 			(at 156.21 127 0)
 			(effects
@@
 	)
 	(symbol
-		(lib_id "Device:L")
+		(lib_id "joka:L")
 		(at 127 118.11 0)
 		(unit 1)
@@
 			)
 		)
-		(property "Footprint" ""
+		(property "Footprint" "joka:L_0805_2012Metric"
 			(at 127 118.11 0)
 			(effects
@@
 	)
 	(symbol
-		(lib_id "Device:Fuse")
+		(lib_id "joka:Fuse")
 		(at 194.31 76.2 90)
 		(unit 1)
@@
 			)
 		)
-		(property "Footprint" ""
+		(property "Footprint" "joka:Fuse_0805_2012Metric"
 			(at 194.31 77.978 90)
 			(effects
@@
 	)
 	(symbol
-		(lib_id "Device:C")
+		(lib_id "joka:C")
 		(at 63.5 118.11 0)
 		(unit 1)
@@
 			)
 		)
-		(property "Footprint" ""
+		(property "Footprint" "joka:C_0805_2012Metric"
 			(at 64.4652 121.92 0)
 			(effects
@@
 	)
 	(symbol
-		(lib_id "Device:L")
+		(lib_id "joka:L")
 		(at 101.6 85.09 0)
 		(unit 1)
@@
 			)
 		)
-		(property "Footprint" ""
+		(property "Footprint" "joka:L_0805_2012Metric"
 			(at 101.6 85.09 0)
 			(effects
@@
 	)
 	(symbol
-		(lib_id "Device:C")
+		(lib_id "joka:C")
 		(at 156.21 63.5 90)
 		(unit 1)
@@
 			)
 		)
-		(property "Footprint" ""
+		(property "Footprint" "joka:C_0805_2012Metric"
 			(at 160.02 62.5348 0)
 			(effects
@@
 	)
 	(symbol
-		(lib_id "Device:R")
+		(lib_id "joka:R")
 		(at 63.5 46.99 0)
 		(unit 1)
@@
 			)
 		)
-		(property "Footprint" ""
+		(property "Footprint" "joka:R_0805_2012Metric"
 			(at 61.722 46.99 90)
 			(effects
@@
 	)
 	(symbol
-		(lib_id "Device:C")
+		(lib_id "joka:C")
 		(at 139.7 111.76 90)
 		(unit 1)
@@
 			)
 		)
-		(property "Footprint" ""
+		(property "Footprint" "joka:C_0805_2012Metric"
 			(at 143.51 110.7948 0)
 			(effects
@@
 	)
 	(symbol
-		(lib_id "Device:L")
+		(lib_id "joka:L")
 		(at 156.21 76.2 90)
 		(unit 1)
@@
 			)
 		)
-		(property "Footprint" ""
+		(property "Footprint" "joka:L_0805_2012Metric"
 			(at 156.21 76.2 0)
 			(effects
@@
 	)
 	(symbol
-		(lib_id "Device:C")
+		(lib_id "joka:C")
 		(at 92.71 76.2 90)
 		(unit 1)
@@
 			)
 		)
-		(property "Footprint" ""
+		(property "Footprint" "joka:C_0805_2012Metric"
 			(at 96.52 75.2348 0)
 			(effects
@@
 	)
 	(symbol
-		(lib_id "Device:R")
+		(lib_id "joka:R")
 		(at 156.21 111.76 90)
 		(unit 1)
@@
 			)
 		)
-		(property "Footprint" ""
+		(property "Footprint" "joka:R_0805_2012Metric"
 			(at 156.21 113.538 90)
 			(effects
@@
 	)
 	(symbol
-		(lib_id "Device:L")
+		(lib_id "joka:L")
 		(at 54.61 127 90)
 		(unit 1)
@@
 			)
 		)
-		(property "Footprint" ""
+		(property "Footprint" "joka:L_0805_2012Metric"
 			(at 54.61 127 0)
 			(effects
@@
 	)
 	(symbol
-		(lib_id "Device:R")
+		(lib_id "joka:R")
 		(at 156.21 91.44 90)
 		(unit 1)
@@
 			)
 		)
-		(property "Footprint" ""
+		(property "Footprint" "joka:R_0805_2012Metric"
 			(at 156.21 93.218 90)
 			(effects
@@
 	)
 	(symbol
-		(lib_id "Device:C")
+		(lib_id "joka:C")
 		(at 156.21 139.7 90)
 		(unit 1)
@@
 			)
 		)
-		(property "Footprint" ""
+		(property "Footprint" "joka:C_0805_2012Metric"
 			(at 160.02 138.7348 0)
 			(effects
@@
 	)
 	(symbol
-		(lib_id "Device:C")
+		(lib_id "joka:C")
 		(at 92.71 127 90)
 		(unit 1)
@@
 			)
 		)
-		(property "Footprint" ""
+		(property "Footprint" "joka:C_0805_2012Metric"
 			(at 96.52 126.0348 0)
 			(effects
@@
 	)
 	(symbol
-		(lib_id "Device:C")
+		(lib_id "joka:C")
 		(at 54.61 38.1 90)
 		(unit 1)
@@
 			)
 		)
-		(property "Footprint" ""
+		(property "Footprint" "joka:C_0805_2012Metric"
 			(at 58.42 37.1348 0)
 			(effects
@@
 	)
 	(symbol
-		(lib_id "Device:C")
+		(lib_id "joka:C")
 		(at 139.7 91.44 90)
 		(unit 1)
@@
 			)
 		)
-		(property "Footprint" ""
+		(property "Footprint" "joka:C_0805_2012Metric"
 			(at 143.51 90.4748 0)
 			(effects
