File: joka.kicad_sch (KiCad schematic)
At the start: 3 parts, among them J1 Conn, J2 ANT1, J3 ANT2

Commit message: intial version of pcb
Parts:
- J1: footprint (none) -> joka:PinSocket_2x05_P2.54mm_Vertical; symbol Connector:Conn_01x10_Pin -> joka:Conn_01x10_Pin
- J2, J3: footprint (none) -> joka:PinSocket_1x01_P2.54mm_Vertical; symbol Connector:Conn_01x01_Socket -> joka:Conn_01x01_Socket
Connections:
- net Reader/IRQ: now also J1.7 (Pin_7); no longer J1.9 (Pin_9)
- net Reader/VEN: now also J1.9 (Pin_9); no longer J1.7 (Pin_7)
Changed lines of the file:
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@@
 	)
 	(symbol
-		(lib_id "Connector:Conn_01x01_Socket")
+		(lib_id "joka:Conn_01x01_Socket")
 		(at 214.63 88.9 0)
 		(unit 1)
@@
 			)
 		)
-		(property "Footprint" ""
+		(property "Footprint" "joka:PinSocket_1x01_P2.54mm_Vertical"
 			(at 214.63 88.9 0)
 			(effects
@@
 	)
 	(symbol
-		(lib_id "Connector:Conn_01x01_Socket")
+		(lib_id "joka:Conn_01x01_Socket")
 		(at 214.63 93.98 0)
 		(unit 1)
@@
 			)
 		)
-		(property "Footprint" ""
+		(property "Footprint" "joka:PinSocket_1x01_P2.54mm_Vertical"
 			(at 214.63 93.98 0)
 			(effects
@@
 	)
 	(symbol
-		(lib_id "Connector:Conn_01x10_Pin")
+		(lib_id "joka:Conn_01x10_Pin")
 		(at 60.96 90.17 0)
 		(unit 1)
@@
 			)
 		)
-		(property "Footprint" ""
+		(property "Footprint" "joka:PinSocket_2x05_P2.54mm_Vertical"
 			(at 60.96 90.17 0)
 			(effects
@@
 		)
 		(pin "VEN" input
-			(at 101.6 93.98 180)
+			(at 101.6 99.06 180)
 			(effects
 				(font
@@
 		)
 		(pin "IRQ" input
-			(at 101.6 99.06 180)
-			(effects
-				(font
+			(at 101.6 93.98 180)
+			(effects
+				(font
