File: reader.kicad_sch (KiCad schematic)
At the start: 13 parts, among them IC1 PN7160B1HN_C100E, Y1 XRCGB27M120F3M10R0

Commit message: intial version of pcb
Parts:
- C1, C2, C3, C4, C5, C6, C7, C8: footprint (none) -> joka:C_0805_2012Metric; symbol Device:C_Small -> joka:C_Small
- C10, C9: footprint (none) -> joka:C_0805_2012Metric; symbol Device:C -> joka:C
- IC1: footprint QFN50P600X600X100-41N-D -> joka:PN7160B1HNC100E
- R1: footprint (none) -> joka:R_0805_2012Metric; symbol Device:R -> joka:R
Changed lines of the file:
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@@
 	)
 	(symbol
-		(lib_id "Device:C_Small")
+		(lib_id "joka:C_Small")
 		(at 96.52 134.62 0)
 		(unit 1)
@@
 			)
 		)
-		(property "Footprint" ""
+		(property "Footprint" "joka:C_0805_2012Metric"
 			(at 96.52 134.62 0)
 			(effects
@@
 	)
 	(symbol
-		(lib_id "Device:C_Small")
+		(lib_id "joka:C_Small")
 		(at 151.13 140.97 0)
 		(unit 1)
@@
 			)
 		)
-		(property "Footprint" ""
+		(property "Footprint" "joka:C_0805_2012Metric"
 			(at 151.13 140.97 0)
 			(effects
@@
 	)
 	(symbol
-		(lib_id "Device:C_Small")
+		(lib_id "joka:C_Small")
 		(at 81.28 60.96 0)
 		(unit 1)
@@
 			)
 		)
-		(property "Footprint" ""
+		(property "Footprint" "joka:C_0805_2012Metric"
 			(at 81.28 60.96 0)
 			(effects
@@
 			)
 		)
-		(property "Footprint" "QFN50P600X600X100-41N-D"
+		(property "Footprint" "joka:PN7160B1HNC100E"
 			(at 151.13 152.07 0)
 			(effects
@@
 	)
 	(symbol
-		(lib_id "Device:C_Small")
+		(lib_id "joka:C_Small")
 		(at 129.54 138.43 0)
 		(unit 1)
@@
 			)
 		)
-		(property "Footprint" ""
+		(property "Footprint" "joka:C_0805_2012Metric"
 			(at 129.54 138.43 0)
 			(effects
@@
 	)
 	(symbol
-		(lib_id "Device:R")
+		(lib_id "joka:R")
 		(at 80.01 91.44 0)
 		(unit 1)
@@
 			)
 		)
-		(property "Footprint" ""
+		(property "Footprint" "joka:R_0805_2012Metric"
 			(at 78.232 91.44 90)
 			(effects
@@
 	)
 	(symbol
-		(lib_id "Device:C")
+		(lib_id "joka:C")
 		(at 212.09 78.74 0)
 		(unit 1)
@@
 			)
 		)
-		(property "Footprint" ""
+		(property "Footprint" "joka:C_0805_2012Metric"
 			(at 213.0552 82.55 0)
 			(effects
@@
 	)
 	(symbol
-		(lib_id "Device:C_Small")
+		(lib_id "joka:C_Small")
 		(at 193.04 101.6 0)
 		(unit 1)
@@
 			)
 		)
-		(property "Footprint" ""
+		(property "Footprint" "joka:C_0805_2012Metric"
 			(at 193.04 101.6 0)
 			(effects
@@
 	)
 	(symbol
-		(lib_id "Device:C")
+		(lib_id "joka:C")
 		(at 196.85 78.74 0)
 		(unit 1)
@@
 			)
 		)
-		(property "Footprint" ""
+		(property "Footprint" "joka:C_0805_2012Metric"
 			(at 197.8152 82.55 0)
 			(effects
@@
 	)
 	(symbol
-		(lib_id "Device:C_Small")
+		(lib_id "joka:C_Small")
 		(at 163.83 140.97 0)
 		(unit 1)
@@
 			)
 		)
-		(property "Footprint" ""
+		(property "Footprint" "joka:C_0805_2012Metric"
 			(at 163.83 140.97 0)
 			(effects
@@
 	)
 	(symbol
-		(lib_id "Device:C_Small")
+		(lib_id "joka:C_Small")
 		(at 180.34 101.6 0)
 		(unit 1)
@@
 			)
 		)
-		(property "Footprint" ""
+		(property "Footprint" "joka:C_0805_2012Metric"
 			(at 180.34 101.6 0)
 			(effects
@@
 	)
 	(symbol
-		(lib_id "Device:C_Small")
+		(lib_id "joka:C_Small")
 		(at 113.03 146.05 0)
 		(unit 1)
@@
 			)
 		)
-		(property "Footprint" ""
+		(property "Footprint" "joka:C_0805_2012Metric"
 			(at 113.03 146.05 0)
 			(effects
